File: PCB/OTThing.kicad_pcb (KiCad board)
At the start: 2 copper layers, 51 x 71 mm, 114 parts, among them IC1 TPS61041, J3 USB_C_Receptacle_USB2.0, K1 G6K-2F-Y-5V, Q1 BC857C, Q10 BC847C, Q11 BC857C, Q12 BC847C, Q13 BC847C, Q2 BC847C, Q4 BC857C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

Commit message: update KiCad libraries
Parts:
- removed FID1, FID2, FID3: Fiducial, Fiducial:Fiducial_0.5mm_Mask1.5mm
