File: PCB/OTThing.kicad_pcb (KiCad board)
At the start: 2 copper layers, 51 x 71 mm, 111 parts, among them IC1 TPS61041, J3 USB_C_Receptacle_USB2.0, K1 G6K-2F-Y-5V, Q1 BC857C, Q10 BC847C, Q11 BC857C, Q12 BC847C, Q13 BC847C, Q2 BC847C, Q4 BC857C, Q5 BC857C, Q6 BC857C, Q7 BC857C, Q8 BC847C, Q9 BC847C, SW1 RST/CONFIG, SW2 BOOT, U1 ESP32-C3-WROOM-02, U5 USBLC6-2SC6, U6 AMS1117-3.3

Commit message: update silkscreen
Routing:
- net /EN24: track 23.8 -> 23.9 mm, vias 2 -> 0
- net GND: vias 107 -> 108
