File: Tester PCB/_restore_backup_2026-09-19T18-04-33-754/OT Thing Tester.kicad_pcb (KiCad board)
At the start: 2 copper layers, 84 x 93 mm, 68 parts, among them J1 Conn_01x05, J2 Conn_01x08, J3 Barrel_Jack_Switch, J4 USB_C_Receptacle_USB2.0, Q1 BSP62, Q2 BSP62, Q3 BC847, Q4 BC857, Q5 BC847, Q6 BC857, U1 LM358, U2 DS18B20, U3 DS18B20

Commit message: Tester PCB layout updates
Parts:
- moved H4 8.00 mm to (175.4, 61.2)
- moved H6 8.00 mm to (175.4, 144.2)
- moved D1 2.00 mm to (166.3, 116.7)
- moved D3 2.00 mm to (166.3, 113.2)
- moved D4 2.00 mm to (166.3, 108.0)
- moved D5 2.00 mm to (166.3, 104.4)
Routing:
- net +3.3V: track 130.7 -> 126.7 mm
- net Net-(D5-K): track 3.90 -> 1.90 mm
- net Net-(D5-A): track 11.3 -> 9.26 mm
- net Net-(D4-K): track 3.90 -> 1.90 mm
- net Net-(D3-K): track 3.90 -> 1.90 mm
- net Net-(D3-A): track 11.3 -> 9.27 mm
- net Net-(D1-K): track 3.90 -> 1.90 mm
Other:
- board size 84 x 93 mm -> 92 x 93 mm
- board text added: "OT Thing Tester - www.seegel-systeme.de - 40/25"
- board text removed: "+28 V"
- board text removed: "OT Thing Tester - www.seegel-systeme.de - 40/26"
