File: Tester PCB/_restore_backup_2026-09-19T18-04-33-754/OT Thing Tester.kicad_sch (KiCad schematic)
At the start: 67 parts, among them J1 Conn_01x05, J2 Conn_01x08, J3 Barrel_Jack_Switch, J4 USB_C_Receptacle_USB2.0, Q1 BSP62, Q2 BSP62, Q3 BC847, Q4 BC857, Q5 BC847, Q6 BC857, U1 LM358, U2 DS18B20, U3 DS18B20

Commit message: Tester PCB layout updates
Parts:
- C1, C2, C3, C4, R1, R10, R11, R12, R13, R14, R15, R16, R17, R18, R2, R3, R4, R5, R6, R7, R8, R9: KiLib_Generator SMD_2terminal_chip_molded -> (none)
- D1, D3, D4, D5: KiLib_Generator 1=K 2=A -> (none)
- H7, H8, H9: KiLib_Generator mounting_hardware/mounting_hole -> (none)
- Q3, Q4, Q5, Q6: KiLib_Generator package/gullwing -> (none)
- RV1, RV2: KiLib_Generator potentiometer/THT -> (none)
